Commit message: 调整多个启动文件中的 odom_frame_id 参数为 odom，新增 EKF 配置项 odom0_differential 和 odom0_relative

File: src/turn_on_wheeltec_robot/urdf/chair_diff_robot.urdf (robot description, URDF)
Before this commit: robot wheeltec_robot, 4 links, 3 joints
Links:
- removed link front_wheel_link
- added link front_left_caster_link
- added link front_left_wheel_link; visual cylinder length=0.02 radius=0.0325
- added link front_right_caster_link
- added link front_right_wheel_link; visual cylinder length=0.02 radius=0.0325
Joints:
- removed joint front_wheel_joint
- added joint front_left_caster_swivel_joint: type continuous, parent base_link, child front_left_caster_link, origin xyz=0.15 0.08 0.0325 rpy=0 0 0, axis 0 0 1
- added joint front_left_caster_wheel_joint: type continuous, parent front_left_caster_link, child front_left_wheel_link, origin xyz=0 0 0 rpy=1.57 0 0, axis 0 1 0
- added joint front_right_caster_swivel_joint: type continuous, parent base_link, child front_right_caster_link, origin xyz=0.15 -0.08 0.0325 rpy=0 0 0, axis 0 0 1
- added joint front_right_caster_wheel_joint: type continuous, parent front_right_caster_link, child front_right_wheel_link, origin xyz=0 0 0 rpy=1.57 0 0, axis 0 1 0
